File: KICAD_files/POWER.kicad_sch (KiCad schematic)
At the start: 103 parts, among them J1 10118193-0001LF, J2 10118193-0001LF, Q1 S8050, Q2 S8050

Commit message: Added
Added
Other:
- note added: "DEBUG"
- note removed: "DEBUGG"
- moved on the sheet: C?, CA?, D1, H1, H2, H3, H4, J1, J2, J?, L?, Q1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
