File: KICAD_files/ETHERNET.kicad_sch (KiCad schematic)
At the start: 42 parts, among them J7 HR911130A1, U10 RTL8211E-VB-CG, Y1 25MHz

Commit message: Added
Added
Other:
- moved on the sheet: C36, C37, C38, C39, C40, C41, C42, C43, C44, C45, C46, C47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
