File: KICAD_files/IO-SDR_Rev_1.0.kicad_sch (KiCad schematic)
At the start: 0 parts

Commit message: Added
Added
Other:
- note added: "- Camera Connector - Onboard sensors - Rounded Edges"
- note added: "2.0 Ideas"
- note added: "IO-SDR_Rev_1.0"
Changed lines of the file:
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@@
 (kicad_sch (version 20230121) (generator eeschema)
   (paper "A3")
+  (text "IO-SDR_Rev_1.0" (at 148.717 101.346 0)
+    (effects (font (face "Verdana") (size 10 10)) (justify left bottom))
+  )
+  (text "2.0 Ideas" (at 20.066 218.44 0)
+    (effects (font (size 4 4)) (justify left bottom))
+  )
+  (text "- Camera Connector\n- Onboard sensors\n- Rounded Edges"
+    (at 17.145 242.57 0)
+    (effects (font (size 4 4)) (justify left bottom))
+  )
   (sheet (at 208.407 121.539) (size 49.276 22.987)
     (stroke (width 0.1524) (type solid))

Commit message: Big Cleanup
Big Cleanup
Other:
- added sheet SENSORS (SENSORS.kicad_sch)
- note added: "- Camera Connector - Onboard sensors (Accel, Mag, Gyro, Barometer, etc.) - Rounded Edges - Time-of-Flight sensor - RTC - Battery - TF card - LCD Screen - PMOD Connectors - Memory Upgrades"
- note removed: "- Camera Connector - Onboard sensors - Rounded Edges"
Changed lines of the file:
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@@
 (kicad_sch (version 20230121) (generator eeschema)
   (paper "A3")
-  (text "IO-SDR_Rev_1.0" (at 148.717 101.346 0)
+  (text "IO-SDR_Rev_1.0" (at 144.78 114.3 0)
     (effects (font (face "Verdana") (size 10 10)) (justify left bottom))
   )
-  (text "2.0 Ideas" (at 20.066 218.44 0)
+  (text "2.0 Ideas" (at 20.066 212.217 0)
     (effects (font (size 4 4)) (justify left bottom))
   )
-  (text "- Camera Connector\n- Onboard sensors\n- Rounded Edges"
-    (at 17.145 242.57 0)
+  (text "- Camera Connector\n- Onboard sensors (Accel, Mag, Gyro, Barometer, etc.)\n- Rounded Edges\n- Time-of-Flight sensor \n- RTC\n- Battery\n- TF card\n- LCD Screen\n- PMOD Connectors \n- Memory Upgrades\n"
+    (at 17.399 277.622 0)
     (effects (font (size 4 4)) (justify left bottom))
   )
-  (sheet (at 208.407 121.539) (size 49.276 22.987)
+  (sheet (at 208.28 121.92) (size 48.26 22.86)
     (stroke (width 0.1524) (type solid))
     (fill (color 0 0 0 0.0000))
-    (property "Sheetname" "AD9361" (at 208.28 121.158 0)
+    (property "Sheetname" "AD9361" (at 208.153 121.539 0)
       (effects (font (size 1.27 1.27)) (justify left bottom))
     )
-    (property "Sheetfile" "AD9361.kicad_sch" (at 208.407 146.2536 0)
+    (property "Sheetfile" "AD9361.kicad_sch" (at 208.28 146.6346 0)
       (effects (font (size 1.27 1.27)) (justify left top))
     )
@@
     )
   )
-  (sheet (at 267.97 121.285) (size 49.403 22.987) (fields_autoplaced)
+  (sheet (at 266.7 121.92) (size 48.26 22.86) (fields_autoplaced)
     (stroke (width 0.1524) (type solid))
     (fill (color 0 0 0 0.0000))
-    (property "Sheetname" "XC7Z010" (at 267.97 120.5734 0)
+    (property "Sheetname" "XC7Z010" (at 266.7 121.2084 0)
       (effects (font (size 1.27 1.27)) (justify left bottom))
     )
-    (property "Sheetfile" "XC7Z010.kicad_sch" (at 267.97 144.8566 0)
+    (property "Sheetfile" "XC7Z010.kicad_sch" (at 266.7 145.4916 0)
       (effects (font (size 1.27 1.27)) (justify left top))
     )
@@
     )
   )
-  (sheet (at 149.352 121.158) (size 48.006 24.511)
+  (sheet (at 91.44 121.92) (size 48.26 22.86)
     (stroke (width 0.1524) (type solid))
     (fill (color 0 0 0 0.0000))
-    (property "Sheetname" "ETHERNET" (at 149.352 120.777 0)
+    (property "Sheetname" "ETHERNET" (at 91.44 121.539 0)
       (effects (font (size 1.27 1.27)) (justify left bottom))
     )
-    (property "Sheetfile" "ETHERNET.kicad_sch" (at 149.479 146.558 0)
+    (property "Sheetfile" "ETHERNET.kicad_sch" (at 91.567 147.32 0)
       (effects (font (size 1.27 1.27)) (justify left top))
     )
@@
     )
   )
-  (sheet (at 91.186 121.539) (size 47.752 24.257) (fields_autoplaced)
+  (sheet (at 149.86 121.92) (size 48.26 22.86) (fields_autoplaced)
     (stroke (width 0.1524) (type solid))
     (fill (color 0 0 0 0.0000))
-    (property "Sheetname" "POWER" (at 91.186 120.8274 0)
+    (property "Sheetname" "POWER" (at 149.86 121.2084 0)
       (effects (font (size 1.27 1.27)) (justify left bottom))
     )
-    (property "Sheetfile" "POWER.kicad_sch" (at 91.186 146.3806 0)
+    (property "Sheetfile" "POWER.kicad_sch" (at 149.86 147.0156 0)
       (effects (font (size 1.27 1.27)) (justify left top))
     )
@@
       )
     )
+  )
+  (sheet (at 91.44 165.1) (size 48.26 22.86)
+    (stroke (width 0.1524) (type solid))
+    (fill (color 0 0 0 0.0000))
+    (property "Sheetname" "SENSORS" (at 91.44 164.719 0)
+      (effects (font (size 1.27 1.27)) (justify left bottom))
+    )
+    (property "Sheetfile" "SENSORS.kicad_sch" (at 91.567 190.5 0)
+      (effects (font (size 1.27 1.27)) (justify left top))
+    )
+    (instances
+      (project "IO-SDR_Rev_1.0"
+        (path "/38786148-0fd1-46d3-8412-9a7876291ebf" (page "5"))
+      )
+    )
